File: hardware/dc-dc/dc-dc.kicad_sch (KiCad schematic)
At the start: 1 part, among them U1 MP8859GQ-0000-P

Commit message: [PCB] Add PCB
Parts:
- added C1: 100u, Capacitor_Tantalum_SMD:CP_EIA-7343-43_Kemet-X_Pad2.25x2.55mm_HandSolder, symbol Device:C_Polarized
- added C10, C11, C12, C13, C14, C2: 22u, Capacitor_SMD:C_1206_3216Metric_Pad1.33x1.80mm_HandSolder, symbol Device:C
- added C3, C7, C8, C9: 100n, Capacitor_SMD:C_0402_1005Metric_Pad0.74x0.62mm_HandSolder, symbol Device:C
- added C4, C5: 22n, Capacitor_SMD:C_0402_1005Metric_Pad0.74x0.62mm_HandSolder, symbol Device:C
- added C6: 1u, Capacitor_SMD:C_0603_1608Metric_Pad1.08x0.95mm_HandSolder, symbol Device:C
- added J1: Conn_01x06, Connector_PinHeader_2.54mm:PinHeader_1x06_P2.54mm_Vertical, symbol Connector_Generic:Conn_01x06
- added J2, J3: Screw_Terminal_01x02, TerminalBlock_Phoenix:TerminalBlock_Phoenix_PT-1,5-2-3.5-H_1x02_P3.50mm_Horizontal, symbol Connector:Screw_Terminal_01x02
- added J4: Raspberry_Pi_2_3, symbol Connector:Raspberry_Pi_2_3
- added L1: 10u, WE-LHMI-7050:IND_7050-WE-LHMI_WRE, symbol Device:L
- added R1, R2: 10k, Resistor_SMD:R_0402_1005Metric_Pad0.72x0.64mm_HandSolder, symbol Device:R
- added R3, R4: 499k, Resistor_SMD:R_0402_1005Metric_Pad0.72x0.64mm_HandSolder, symbol Device:R
- added R5: 301k, Resistor_SMD:R_0402_1005Metric_Pad0.72x0.64mm_HandSolder, symbol Device:R
- added R6: 21k5, Resistor_SMD:R_0402_1005Metric_Pad0.72x0.64mm_HandSolder, symbol Device:R
- added R7, R8: 0, Resistor_SMD:R_0402_1005Metric_Pad0.72x0.64mm_HandSolder, symbol Device:R
- added R9: 100k, Resistor_SMD:R_0402_1005Metric_Pad0.72x0.64mm_HandSolder, symbol Device:R
- U1: footprint QFN-16_MP8859_00_MNP -> MP8859:QFN-16_MP8859_00_MNP
Connections:
- net IN: now reaches U1.1 (IN)
- net IN: now also C1.1, C2.1, C3.1, J3.1 (Pin_1), R3.1
- net GND: now reaches U1.10 (AGND)
- net GND: now also U1.11 (GND), U1.2 (GND), C1.2, C10.2, C11.2, C12.2, C13.2, C14.2, C2.2, C3.2, C4.2, C5.2, C6.2, C9.2, J1.2 (Pin_2), J1.3 (Pin_3), J2.1 (Pin_1), J3.2 (Pin_2), J4.14 (GND), J4.20 (GND), J4.25 (GND), J4.30 (GND), J4.34 (GND), J4.39 (GND), J4.6 (GND), J4.9 (GND), R5.2, R6.2
- net OUT: now reaches U1.12 (OUT)
- net OUT: now also C10.1, C11.1, C12.1, C13.1, C14.1, C9.1, J2.2 (Pin_2)
- net at U1.13 (BST2): now also R8.1
- net at U1.14 (SW2): now also C8.2, L1.1
- net at U1.15 (SW1): now also C7.1, L1.2
- net at U1.16 (BST1): now also R7.1
- net at U1.3 (EN): now also C4.1, R3.2
- net at U1.4 (ADD): now also R4.2, R5.1
- net SCL: now reaches U1.5 (SCL)
- net SCL: now also J1.4 (Pin_4), J4.5 (SCL/GPIO3), R1.2
- net SDA: now reaches U1.6 (SDA)
- net SDA: now also J1.5 (Pin_5), J4.3 (SDA/GPIO2), R2.2
- net at U1.7 (OC): now also C5.1, R6.1
- net ALT: now reaches U1.8 (ALT)
- net ALT: now also J1.6 (Pin_6), J4.7 (GCLK0/GPIO4), R9.1
- net VCC: now reaches U1.9 (VCC)
- net VCC: now also C6.1, J1.1 (Pin_1), R1.1, R2.1, R4.1, R9.2
- new net: C8.1, R8.2
- new net: C7.2, R7.2
- no-connect marks 0 -> 29
Other:
- note added: "1-12V"
- note added: "2.8-22V"
- note added: "КОНЕКТОРИ"
- note added: "ПОНИЖАВАЩО-ПОВИШАВАЩ ПРЕОБРАЗУВАТЕЛ"
- company: (none) -> Петър Николов
- title: (none) -> Buck-Boost захранване, управлявано с RaspberryPi
- moved on the sheet: U1

Commit message: [Schematic/PCB] Add qwiic connector and 2 electrolytic caps
Parts:
- removed J1: Conn_01x06, Connector_PinHeader_2.54mm:PinHeader_1x06_P2.54mm_Vertical, symbol Connector_Generic:Conn_01x06
- removed R1, R2: 10k, Resistor_SMD:R_0402_1005Metric_Pad0.72x0.64mm_HandSolder, symbol Device:R
- added C1, C16: 100u, Capacitor_SMD:CP_Elec_6.3x7.7, symbol Device:C_Polarized
- added J1: PRT-14417, QWIIC:SPARKFUN_PRT-14417, symbol QWIIC:PRT-14417
- renumbered C9 to C10, C10 to C11, C11 to C12, C12 to C13, C13 to C14, C14 to C15, C1 to C2, C2 to C3, C3 to C4, C4 to C5, C5 to C6, C6 to C7, C7 to C8, C8 to C9, R3 to R1, R4 to R2, R5 to R3, R6 to R4, R9 to R5, R7 to R6, R8 to R7
Connections:
- net GND: now also C1.2, C16.2, J1.4
- net IN: now also C1.1
- net OUT: now also C16.1
- net SCL: now also J1.1
- net SDA: now also J1.2
- no-connect marks 29 -> 30
Other:
- moved on the sheet: C10, C11, C12, C13, C14, C15, C2, C3, C4, C5, C6, C7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
